File: STM32-V1/STM32-V1.kicad_pcb (KiCad board)
At the start: 4 copper layers, 50 x 54 mm, 48 parts, among them J1 USB_B_Micro, J2 Conn_02x03_Odd_Even, SW1 SW_SPDT, U1 LD1086D2T33TR, U2 USBLC6-2SC6, U3 BMP280, U4 Ai-Thinker-Ra-02, U5 MPU-6050, U6 STM32F103C8Tx, U7 CH340E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

Commit message: My first KiCad Design, This is Rev 1
Parts:
- F1: value JK-nSMD110-SF -> JK-nSMD150-SF
