File: STM32-V1/STM32-V1.sch (KiCad schematic (older format))
At the start: 47 parts, among them J1 USB_B_Micro, J2 Conn_02x03_Odd_Even, SW1 SW_SPDT, U1 LD1086D2T33TR, U2 USBLC6-2SC6, U3 BMP280, U4 Ai-Thinker-Ra-02, U5 MPU-6050, U6 STM32F103C8Tx, U7 CH340E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

Commit message: My first KiCad Design, This is Rev 1
Parts:
- C1, C2: LSCS Part # (none) -> C108529
- C10: LSCS Part # (none) -> C15195
- C11, C12, C13, C14, C18, C19, C4, C5, C6, C7: LSCS Part # (none) -> C1525
- C15: LSCS Part # (none) -> C1531
- C16, C17: LSCS Part # (none) -> C22397
- C3: LSCS Part # (none) -> C19666
- C8: LSCS Part # (none) -> C29266
- C9: LSCS Part # (none) -> C15525
- D1, D3: LSCS Part # (none) -> C2286
- D2: LSCS Part # (none) -> C72041
- F1: value JK-nSMD110-SF -> JK-nSMD150-SF; LSCS Part # (none) -> C369553
- J1: LSCS Part # (none) -> C136000
- L1: LSCS Part # (none) -> C18830
- R1, R6: LSCS Part # (none) -> C21190
- R2: LSCS Part # (none) -> C25804
- R3: LSCS Part # (none) -> C22843
- R4, R5, R7, R8: LSCS Part # (none) -> C25933
- U1: LSCS Part # (none) -> C7915
- U2: LSCS Part # (none) -> C7519
- U3: LSCS Part # (none) -> C83291
- U4: LSCS Part # (none) -> C90039
- U5: LSCS Part # (none) -> MPU-6050
- U6: LSCS Part # (none) -> C8734
- U7: LSCS Part # (none) -> C99652
- Y1: LSCS Part # (none) -> C251585
Changed lines of the file:
@@
 F 2 "Package_TO_SOT_SMD:TO-263-2" H 6525 1850 50  0001 C CNN
 F 3 "https://www.st.com/resource/en/datasheet/ld1086.pdf" H 6525 1850 50  0001 C CNN
+F 4 "C7915" H 6525 1350 50  0001 C CNN "LSCS Part #"
 	1    6525 1350
 	1    0    0    -1
@@
 F 2 "Capacitor_SMD:C_0603_1608Metric" H 700 3150 50  0001 C CNN
 F 3 "~" H 700 3150 50  0001 C CNN
+F 4 "C19666" H 700 3150 50  0001 C CNN "LSCS Part #"
 	1    700  3150
 	1    0    0    -1
@@
 F 2 "Capacitor_SMD:C_0402_1005Metric" H 1025 3150 50  0001 C CNN
 F 3 "~" H 1025 3150 50  0001 C CNN
+F 4 "C1525" H 1025 3150 50  0001 C CNN "LSCS Part #"
 	1    1025 3150
 	1    0    0    -1
@@
 F 2 "Capacitor_SMD:C_0402_1005Metric" H 1375 3150 50  0001 C CNN
 F 3 "~" H 1375 3150 50  0001 C CNN
+F 4 "C1525" H 1375 3150 50  0001 C CNN "LSCS Part #"
 	1    1375 3150
 	1    0    0    -1
@@
 F 2 "Capacitor_SMD:C_0402_1005Metric" H 1725 3150 50  0001 C CNN
 F 3 "~" H 1725 3150 50  0001 C CNN
+F 4 "C1525" H 1725 3150 50  0001 C CNN "LSCS Part #"
 	1    1725 3150
 	1    0    0    -1
@@
 F 2 "Capacitor_SMD:C_0402_1005Metric" H 3700 3150 50  0001 C CNN
 F 3 "~" H 3700 3150 50  0001 C CNN
+F 4 "C15525" H 3700 3150 50  0001 C CNN "LSCS Part #"
 	1    3700 3150
 	1    0    0    -1
@@
 F 2 "Capacitor_SMD:C_0402_1005Metric" H 3400 3150 50  0001 C CNN
 F 3 "~" H 3400 3150 50  0001 C CNN
+F 4 "C29266" H 3400 3150 50  0001 C CNN "LSCS Part #"
 	1    3400 3150
 	1    0    0    -1
@@
 F 2 "Inductor_SMD:L_0402_1005Metric" H 3150 3025 50  0001 C CNN
 F 3 "~" H 3150 3025 50  0001 C CNN
+F 4 "C18830" H 3150 3025 50  0001 C CNN "LSCS Part #"
 	1    3150 3025
 	0    -1   -1   0
@@
 F 2 "Resistor_SMD:R_0603_1608Metric" H 3975 4300 50  0001 C CNN
 F 3 "~" H 3975 4300 50  0001 C CNN
+F 4 "C25804" H 3975 4300 50  0001 C CNN "LSCS Part #"
 	1    3975 4300
 	0    1    1    0
@@
 F 2 "Package_QFP:LQFP-48_7x7mm_P0.5mm" H 1750 4425 50  0001 R CNN
 F 3 "http://www.st.com/st-web-ui/static/active/en/resource/technical/document/datasheet/CD00161566.pdf" H 2350 5825 50  0001 C CNN
+F 4 "C8734" H 2350 5825 50  0001 C CNN "LSCS Part #"
 	1    2350 5825
 	1    0    0    -1
@@
 F 2 "Capacitor_SMD:C_0603_1608Metric" H 675 5550 50  0001 C CNN
 F 3 "~" H 675 5550 50  0001 C CNN
+F 4 "C22397" H 675 5550 50  0001 C CNN "LSCS Part #"
 	1    675  5550
 	1    0    0    -1
@@
 F 2 "Capacitor_SMD:C_0603_1608Metric" H 1075 5550 50  0001 C CNN
 F 3 "~" H 1075 5550 50  0001 C CNN
+F 4 "C22397" H 1075 5550 50  0001 C CNN "LSCS Part #"
 	1    1075 5550
 	1    0    0    -1
@@
 F 2 "Resistor_SMD:R_0402_1005Metric" H 4275 6200 50  0001 C CNN
 F 3 "~" H 4275 6200 50  0001 C CNN
+F 4 "C25933" H 4275 6200 50  0001 C CNN "LSCS Part #"
 	1    4275 6200
 	0    1    1    0
@@
 F 2 "Resistor_SMD:R_0402_1005Metric" H 4275 6525 50  0001 C CNN
 F 3 "~" H 4275 6525 50  0001 C CNN
+F 4 "C25933" H 4275 6525 50  0001 C CNN "LSCS Part #"
 	1    4275 6525
 	0    1    1    0
@@
 F 2 "Resistor_SMD:R_0402_1005Metric" H 4275 6875 50  0001 C CNN
 F 3 "~" H 4275 6875 50  0001 C CNN
+F 4 "C25933" H 4275 6875 50  0001 C CNN "LSCS Part #"
 	1    4275 6875
 	0    1    1    0
@@
 F 2 "Resistor_SMD:R_0402_1005Metric" H 4275 7200 50  0001 C CNN
 F 3 "~" H 4275 7200 50  0001 C CNN
+F 4 "C25933" H 4275 7200 50  0001 C CNN "LSCS Part #"
 	1    4275 7200
 	0    1    1    0
@@
 F 2 "Package_TO_SOT_SMD:SOT-23-6" H 3325 875 50  0001 C CNN
 F 3 "https://www.st.com/resource/en/datasheet/usblc6-2.pdf" H 3525 1725 50  0001 C CNN
+F 4 "C7519" H 3325 1375 50  0001 C CNN "LSCS Part #"
 	1    3325 1375
 	1    0    0    -1
@@
 F 2 "Capacitor_Tantalum_SMD:CP_EIA-3216-18_Kemet-A" H 7125 1550 50  0001 C CNN
 F 3 "~" H 7125 1550 50  0001 C CNN
+F 4 "C108529" H 7125 1550 50  0001 C CNN "LSCS Part #"
 	1    7125 1550
 	1    0    0    -1
@@
 F 2 "Capacitor_Tantalum_SMD:CP_EIA-3216-18_Kemet-A" H 5875 1550 50  0001 C CNN
 F 3 "~" H 5875 1550 50  0001 C CNN
+F 4 "C108529" H 5875 1550 50  0001 C CNN "LSCS Part #"
 	1    5875 1550
 	1    0    0    -1
@@
 P 5375 1350
 F 0 "F1" V 5170 1350 50  0000 C CNN
-F 1 "JK-nSMD110-SF" V 5261 1350 50  0000 C CNN
+F 1 "JK-nSMD150-SF" V 5261 1350 50  0000 C CNN
 F 2 "Fuse:Fuse_1206_3216Metric" H 5425 1150 50  0001 L CNN
 F 3 "~" H 5375 1350 50  0001 C CNN
+F 4 "C369553" H 5375 1350 50  0001 C CNN "LSCS Part #"
 	1    5375 1350
 	0    1    1    0
@@
 F 2 "Resistor_SMD:R_0603_1608Metric" H 4200 5350 50  0001 C CNN
 F 3 "~" H 4200 5350 50  0001 C CNN
+F 4 "C22843" H 4200 5350 50  0001 C CNN "LSCS Part #"
 	1    4200 5350
 	1    0    0    -1
@@
 F 2 "LED_SMD:LED_0603_1608Metric" V 4200 5550 50  0001 C CNN
 F 3 "~" V 4200 5550 50  0001 C CNN
+F 4 "C72041" H 4200 5550 50  0001 C CNN "LSCS Part #"
 	1    4200 5550
 	0    -1   -1   0
@@
 F 2 "LED_SMD:LED_0603_1608Metric" V 7575 1500 50  0001 C CNN
 F 3 "~" V 7575 1500 50  0001 C CNN
+F 4 "C2286" H 7575 1500 50  0001 C CNN "LSCS Part #"
 	1    7575 1500
 	0    -1   -1   0
@@
 F 2 "Package_LGA:Bosch_LGA-8_2x2.5mm_P0.65mm_ClockwisePinNumbering" H 9425 2850 50  0001 C CNN
 F 3 "https://ae-bst.resource.bosch.com/media/_tech/media/datasheets/BST-BMP280-DS001.pdf" H 9425 3550 50  0001 C CNN
+F 4 "C83291" H 9425 3550 50  0001 C CNN "LSCS Part #"
 	1    9425 3550
 	1    0    0    -1
@@
 F 2 "Capacitor_SMD:C_0402_1005Metric" H 7200 4525 50  0001 C CNN
 F 3 "~" H 7200 4525 50  0001 C CNN
+F 4 "C1531" H 7200 4525 50  0001 C CNN "LSCS Part #"
 	1    7200 4525
 	1    0    0    -1
@@
 F 2 "Capacitor_SMD:C_0402_1005Metric" H 6775 4525 50  0001 C CNN
 F 3 "~" H 6775 4525 50  0001 C CNN
+F 4 "C1525" H 6775 4525 50  0001 C CNN "LSCS Part #"
 	1    6775 4525
 	1    0    0    -1
@@
 F 2 "Sensor_Motion:InvenSense_QFN-24_4x4mm_P0.5mm" H 6000 3250 50  0001 C CNN
 F 3 "https://store.invensense.com/datasheets/invensense/MPU-6050_DataSheet_V3%204.pdf" H 6000 3900 50  0001 C CNN
+F 4 "MPU-6050" H 6000 4050 50  0001 C CNN "LSCS Part #"
 	1    6000 4050
 	1    0    0    -1
@@
 F 2 "LED_SMD:LED_0603_1608Metric" V 5675 6900 50  0001 C CNN
 F 3 "~" V 5675 6900 50  0001 C CNN
+F 4 "C2286" H 5675 6900 50  0001 C CNN "LSCS Part #"
 	1    5675 6900
 	0    -1   -1   0
@@
 F 2 "Resistor_SMD:R_0603_1608Metric" H 5675 6700 50  0001 C CNN
 F 3 "~" H 5675 6700 50  0001 C CNN
+F 4 "C21190" H 5675 6700 50  0001 C CNN "LSCS Part #"
 	1    5675 6700
 	1    0    0    -1
@@
 F 2 "Capacitor_SMD:C_0402_1005Metric" H 5000 6100 50  0001 C CNN
 F 3 "~" H 5000 6100 50  0001 C CNN
+F 4 "C1525" H 5000 6100 50  0001 C CNN "LSCS Part #"
 	1    5000 6100
 	1    0    0    -1
@@
 F 2 "Capacitor_SMD:C_0402_1005Metric" H 5325 6100 50  0001 C CNN
 F 3 "~" H 5325 6100 50  0001 C CNN
+F 4 "C1525" H 5325 6100 50  0001 C CNN "LSCS Part #"
 	1    5325 6100
 	1    0    0    -1
@@
 F 2 "RF_Module:Ai-Thinker-Ra-02-LoRa" H 10600 1775 50  0001 C CNN
 F 3 "https://docs.ai-thinker.com/_media/lora/docs/c048ps01a1_ra-02_product_specification_v1.1.pdf" H 9600 3775 50  0001 C CNN
+F 4 "C90039" H 9600 3775 50  0001 C CNN "LSCS Part #"
 	1    9600 3775
 	1    0    0    -1
@@
 F 2 "Capacitor_SMD:C_0402_1005Metric" H 8375 3000 50  0001 C CNN
 F 3 "~" H 8375 3000 50  0001 C CNN
+F 4 "C1525" H 8375 3000 50  0001 C CNN "LSCS Part #"
 	1    8375 3000
 	1    0    0    -1
@@
 F 2 "Capacitor_SMD:C_0402_1005Metric" H 10225 2975 50  0001 C CNN
 F 3 "~" H 10225 2975 50  0001 C CNN
+F 4 "C1525" H 10225 2975 50  0001 C CNN "LSCS Part #"
 	1    10225 2975
 	1    0    0    -1
@@
 F 2 "Capacitor_SMD:C_0402_1005Metric" H 5550 2800 50  0001 C CNN
 F 3 "~" H 5550 2800 50  0001 C CNN
+F 4 "C15195" H 5550 2800 50  0001 C CNN "LSCS Part #"
 	1    5550 2800
 	1    0    0    -1
@@
 F 2 "Capacitor_SMD:C_0402_1005Metric" H 6450 2800 50  0001 C CNN
 F 3 "~" H 6450 2800 50  0001 C CNN
+F 4 "C1525" H 6450 2800 50  0001 C CNN "LSCS Part #"
 	1    6450 2800
 	1    0    0    -1
@@
 F 2 "Connector_USB:USB_Micro-B_Molex-105017-0001" H 1125 1300 50  0001 C CNN
 F 3 "~" H 1125 1300 50  0001 C CNN
+F 4 "C136000" H 975 1350 50  0001 C CNN "LSCS Part #"
 	1    975  1350
 	1    0    0    -1
@@
 F 2 "Package_SO:MSOP-10_3x3mm_P0.5mm" H 6350 5850 50  0001 L CNN
 F 3 "https://www.mpja.com/download/35227cpdata.pdf" H 5950 7200 50  0001 C CNN
+F 4 "C99652" H 6300 6400 50  0001 C CNN "LSCS Part #"
 	1    6300 6400
 	1    0    0    -1
@@
 F 2 "Capacitor_SMD:C_0402_1005Metric" H 2075 3150 50  0001 C CNN
 F 3 "~" H 2075 3150 50  0001 C CNN
+F 4 "C1525" H 2075 3150 50  0001 C CNN "LSCS Part #"
 	1    2075 3150
 	1    0    0    -1
@@
 F 2 "Resistor_SMD:R_0603_1608Metric" H 7575 1750 50  0001 C CNN
 F 3 "~" H 7575 1750 50  0001 C CNN
+F 4 "C21190" H 7575 1750 50  0001 C CNN "LSCS Part #"
 	1    7575 1750
 	1    0    0    -1
@@
 F 2 "Crystal:Crystal_SMD_5032-2Pin_5.0x3.2mm" H 875 5275 50  0001 C CNN
 F 3 "~" H 875 5275 50  0001 C CNN
+F 4 "C251585" H 875 5275 50  0001 C CNN "LSCS Part #"
 	1    875  5275
 	1    0    0    -1
